File: BenchTest/BenchTester/BenchTester.kicad_pcb (KiCad board)
At the start: 2 copper layers, 38 parts, among them J1 Conn_01x01_Socket, J2 Conn_01x01_Socket, J3 Conn_01x01_Socket, J4 Conn_01x02_Socket, J5 Conn_01x01_Socket, J6 Conn_01x01_Socket, J7 Conn_01x01_Socket, J8 Conn_01x01_Socket, J9 Conn_01x01_Socket, Q1 Q_NMOS_GDS, Q2 Q_NMOS_GDS, Q3 Q_NMOS_GDS, Q5 Q_NMOS_GDS

Commit message: Board Layout
Routing:
- net /Vdrive: track 203.7 -> 203.1 mm
Other:
- board outline added: 66 x 63.8 mm
Changed lines of the file:
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@@
 		)
+	)
+	(gr_line
+		(start 227.838 50.038)
+		(end 223.774 50.038)
+		(stroke
+			(width 0.05)
+			(type default)
+		)
+		(layer "Edge.Cuts")
+	)
+	(gr_line
+		(start 161.798 50.038)
+		(end 223.774 50.038)
+		(stroke
+			(width 0.05)
+			(type default)
+		)
+		(layer "Edge.Cuts")
+	)
+	(gr_line
+		(start 176.022 113.792)
+		(end 227.838 113.792)
+		(stroke
+			(width 0.05)
+			(type default)
+		)
+		(layer "Edge.Cuts")
+	)
+	(gr_line
+		(start 176.022 113.792)
+		(end 161.798 113.792)
+		(stroke
+			(width 0.05)
+			(type default)
+		)
+		(layer "Edge.Cuts")
+	)
+	(gr_line
+		(start 227.838 113.792)
+		(end 227.838 50.038)
+		(stroke
+			(width 0.05)
+			(type default)
+		)
+		(layer "Edge.Cuts")
+	)
+	(gr_line
+		(start 161.798 113.792)
+		(end 161.798 50.038)
+		(stroke
+			(width 0.05)
+			(type default)
+		)
+		(layer "Edge.Cuts")
 	)
 	(segment
@@
 	)
 	(segment
+		(start 167.031 62.731)
+		(end 168.148 63.848)
+		(width 0.5)
+		(layer "F.Cu")
+		(net 9)
+	)
+	(segment
+		(start 216.408 107.696)
+		(end 220.405999 107.696)
+		(width 0.5)
+		(layer "F.Cu")
+		(net 9)
+	)
+	(segment
 		(start 214.884 112.522)
 		(end 214.884 108.712)
@@
 	)
 	(segment
-		(start 167.031 62.731)
-		(end 168.148 63.848)
-		(width 0.5)
-		(layer "F.Cu")
-		(net 9)
-	)
-	(segment
-		(start 216.408 107.696)
-		(end 220.405999 107.696)
-		(width 0.5)
-		(layer "F.Cu")
-		(net 9)
-	)
-	(segment
-		(start 163.479999 106.583999)
-		(end 170.942 114.046)
+		(start 170.18 113.284)
+		(end 214.122 113.284)
+		(width 0.5)
+		(layer "F.Cu")
+		(net 9)
+	)
+	(segment
+		(start 214.122 113.284)
+		(end 214.884 112.522)
 		(width 0.5)
 		(layer "F.Cu")
@@
 	(segment
 		(start 163.479999 94.645999)
+		(end 163.479999 106.583999)
+		(width 0.5)
+		(layer "F.Cu")
+		(net 9)
+	)
+	(segment
+		(start 163.479999 94.645999)
 		(end 163.479999 66.282001)
+		(width 0.5)
+		(layer "F.Cu")
+		(net 9)
+	)
+	(segment
+		(start 215.9 107.696)
+		(end 216.408 107.696)
+		(width 0.5)
+		(layer "F.Cu")
+		(net 9)
+	)
+	(segment
+		(start 214.884 108.712)
+		(end 215.9 107.696)
 		(width 0.5)
 		(layer "F.Cu")
@@
 	)
 	(segment
-		(start 216.408 107.696)
-		(end 215.9 107.696)
-		(width 0.5)
-		(layer "F.Cu")
-		(net 9)
-	)
-	(segment
-		(start 170.942 114.046)
-		(end 213.36 114.046)
-		(width 0.5)
-		(layer "F.Cu")
-		(net 9)
-	)
-	(segment
 		(start 219.481311 56.921311)
 		(end 213.614 51.054)
@@
 	)
 	(segment
-		(start 213.36 114.046)
-		(end 214.884 112.522)
-		(width 0.5)
-		(layer "F.Cu")
-		(net 9)
-	)
-	(segment
 		(start 167.031 58.171)
 		(end 167.031 62.731)
@@
 	)
 	(segment
-		(start 215.9 107.696)
-		(end 214.884 108.712)
-		(width 0.5)
-		(layer "F.Cu")
-		(net 9)
-	)
-	(segment
 		(start 213.614 51.054)
 		(end 174.148 51.054)
@@
 	)
 	(segment
-		(start 163.479999 94.645999)
-		(end 163.479999 106.583999)
-		(width 0.5)
-		(layer "F.Cu")
+		(start 163.479999 106.583999)
+		(end 170.18 113.284)
+		(width 0.5)
+		(layer "F.Cu")
