File: BenchTest/BenchTester/BenchTester.kicad_pcb (KiCad board)
At the start: 2 copper layers, 66 x 63.8 mm, 38 parts, among them J1 Conn_01x01_Socket, J2 Conn_01x01_Socket, J3 Conn_01x01_Socket, J4 Conn_01x02_Socket, J5 Conn_01x01_Socket, J6 Conn_01x01_Socket, J7 Conn_01x01_Socket, J8 Conn_01x01_Socket, J9 Conn_01x01_Socket, Q1 Q_NMOS_GDS, Q2 Q_NMOS_GDS, Q3 Q_NMOS_GDS, Q5 Q_NMOS_GDS

Commit message: Post DRC
Routing:
- net /Vdrive: track 203.1 -> 203.9 mm
Changed lines of the file:
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@@
-	)
-	(segment
-		(start 166.436001 104.768)
-		(end 166.37 104.834001)
-		(width 0.5)
-		(layer "B.Cu")
-		(net 8)
 	)
 	(segment
@@
 	)
 	(segment
+		(start 215.646 112.776)
+		(end 170.688 112.776)
+		(width 0.5)
+		(layer "B.Cu")
+		(net 8)
+	)
+	(segment
 		(start 167.132 93.472)
 		(end 167.132 97.335998)
@@
 	)
 	(segment
-		(start 215.138 113.284)
-		(end 216.408 112.014)
-		(width 0.5)
-		(layer "B.Cu")
-		(net 8)
-	)
-	(segment
 		(start 224.536 95.504)
 		(end 224.536 69.023272)
@@
 	)
 	(segment
-		(start 216.408 112.014)
-		(end 216.408 110.236)
-		(width 0.5)
-		(layer "B.Cu")
-		(net 8)
-	)
-	(segment
 		(start 172.466 69.596)
 		(end 172.466 68.58)
@@
 	)
 	(segment
+		(start 166.37 108.458)
+		(end 166.37 104.834001)
+		(width 0.5)
+		(layer "B.Cu")
+		(net 8)
+	)
+	(segment
 		(start 221.741999 107.107999)
 		(end 221.741999 99.822001)
@@
 	)
 	(segment
+		(start 216.408 112.014)
+		(end 215.646 112.776)
+		(width 0.5)
+		(layer "B.Cu")
+		(net 8)
+	)
+	(segment
+		(start 216.408 110.236)
+		(end 216.408 112.014)
+		(width 0.5)
+		(layer "B.Cu")
+		(net 8)
+	)
+	(segment
 		(start 167.132 97.335998)
 		(end 167.452001 97.655999)
@@
 	)
 	(segment
-		(start 166.37 104.834001)
-		(end 166.37 108.204)
-		(width 0.5)
-		(layer "B.Cu")
-		(net 8)
-	)
-	(segment
 		(start 178.816 51.054)
 		(end 209.042 51.054)
@@
 	)
 	(segment
-		(start 171.45 113.284)
-		(end 215.138 113.284)
-		(width 0.5)
-		(layer "B.Cu")
-		(net 8)
-	)
-	(segment
 		(start 214.072755 61.418755)
 		(end 215.138 62.484)
@@
 	)
 	(segment
-		(start 166.37 108.204)
-		(end 171.45 113.284)
+		(start 166.37 104.834001)
+		(end 166.436001 104.768)
+		(width 0.5)
+		(layer "B.Cu")
+		(net 8)
+	)
+	(segment
+		(start 170.688 112.776)
+		(end 166.37 108.458)
 		(width 0.5)
 		(layer "B.Cu")
@@
 	)
 	(segment
-		(start 214.884 112.522)
-		(end 214.884 108.712)
-		(width 0.5)
-		(layer "F.Cu")
-		(net 9)
-	)
-	(segment
-		(start 170.18 113.284)
-		(end 214.122 113.284)
-		(width 0.5)
-		(layer "F.Cu")
-		(net 9)
-	)
-	(segment
-		(start 214.122 113.284)
+		(start 214.884 108.712)
 		(end 214.884 112.522)
 		(width 0.5)
@@
 	)
 	(segment
+		(start 214.63 112.776)
+		(end 167.64 112.776)
+		(width 0.5)
+		(layer "F.Cu")
+		(net 9)
+	)
+	(segment
 		(start 219.481311 64.184956)
 		(end 222.705719 67.409364)
@@
 	(segment
 		(start 163.479999 94.645999)
-		(end 163.479999 106.583999)
-		(width 0.5)
-		(layer "F.Cu")
-		(net 9)
-	)
-	(segment
-		(start 163.479999 94.645999)
 		(end 163.479999 66.282001)
-		(width 0.5)
-		(layer "F.Cu")
-		(net 9)
-	)
-	(segment
-		(start 215.9 107.696)
-		(end 216.408 107.696)
-		(width 0.5)
-		(layer "F.Cu")
-		(net 9)
-	)
-	(segment
-		(start 214.884 108.712)
-		(end 215.9 107.696)
 		(width 0.5)
 		(layer "F.Cu")
@@
 	)
 	(segment
+		(start 167.64 112.776)
+		(end 163.479999 108.615999)
+		(width 0.5)
+		(layer "F.Cu")
+		(net 9)
+	)
+	(segment
+		(start 215.9 107.696)
+		(end 214.884 108.712)
+		(width 0.5)
+		(layer "F.Cu")
+		(net 9)
+	)
+	(segment
 		(start 220.472 105.939999)
 		(end 220.758 105.653999)
@@
 	)
 	(segment
+		(start 216.408 107.696)
+		(end 215.9 107.696)
+		(width 0.5)
+		(layer "F.Cu")
+		(net 9)
+	)
+	(segment
 		(start 167.031 58.171)
 		(end 167.031 62.731)
@@
 	)
 	(segment
+		(start 163.479999 108.615999)
+		(end 163.479999 94.645999)
+		(width 0.5)
+		(layer "F.Cu")
+		(net 9)
+	)
+	(segment
 		(start 213.614 51.054)
 		(end 174.148 51.054)
@@
 	)
 	(segment
-		(start 163.479999 106.583999)
-		(end 170.18 113.284)
-		(width 0.5)
-		(layer "F.Cu")
+		(start 214.884 112.522)
+		(end 214.63 112.776)
+		(width 0.5)
+		(layer "F.Cu")
