File: ErrorDisplay/BottomIndicators/ButtomIndicator/ButtomIndicator.kicad_pcb (KiCad board)
At the start: 2 copper layers, 0 parts

Commit message: Board Outline Lain out, needs testing.
Other:
- board outline added: 163.3 x 15 mm
Changed lines of the file:
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@@
 	(net 0 "")
 	(gr_line
-		(start 185.6 100.9)
-		(end 185.6 115.9)
-		(stroke
-			(width 0.05)
-			(type default)
-		)
-		(layer "User.1")
-	)
-	(gr_line
-		(start 187.9 100.9)
-		(end 187.9 115.9)
+		(start 67.2 100.9)
+		(end 230.5 100.9)
+		(stroke
+			(width 0.05)
+			(type default)
+		)
+		(layer "Edge.Cuts")
+	)
+	(gr_line
+		(start 67.2 115.9)
+		(end 67.2 100.9)
+		(stroke
+			(width 0.05)
+			(type default)
+		)
+		(layer "Edge.Cuts")
+	)
+	(gr_line
+		(start 230.5 100.9)
+		(end 230.5 115.9)
+		(stroke
+			(width 0.05)
+			(type default)
+		)
+		(layer "Edge.Cuts")
+	)
+	(gr_line
+		(start 230.5 115.9)
+		(end 67.2 115.9)
+		(stroke
+			(width 0.05)
+			(type default)
+		)
+		(layer "Edge.Cuts")
+	)
+	(gr_line
+		(start 185.1 100.9)
+		(end 185.1 115.9)
+		(stroke
+			(width 0.05)
+			(type default)
+		)
+		(layer "User.1")
+	)
+	(gr_line
+		(start 187.5 100.9)
+		(end 187.5 115.9)
 		(stroke
 			(width 0.05)
@@
 	(gr_line
 		(start 67.2 115.9)
-		(end 236.2 115.9)
+		(end 230.5 115.9)
 		(stroke
 			(width 0.05)
@@
 	(gr_line
 		(start 67.2 100.9)
-		(end 236.2 100.9)
-		(stroke
-			(width 0.05)
-			(type default)
-		)
-		(layer "User.1")
-	)
-	(gr_line
-		(start 236.2 97)
-		(end 236.2 115.7)
-		(stroke
-			(width 0.05)
-			(type default)
-		)
-		(layer "User.1")
-	)
-	(gr_line
-		(start 67.2 97)
-		(end 67.2 115.9)
-		(stroke
-			(width 0.05)
-			(type default)
-		)
-		(layer "User.1")
+		(end 230.5 100.9)
+		(stroke
+			(width 0.05)
+			(type default)
+		)
+		(layer "User.1")
+	)
+	(gr_rect
+		(start 170.6 100.9)
+		(end 185.1 115.9)
+		(stroke
+			(width 0.1)
+			(type default)
+		)
+		(fill none)
+		(layer "User.2")
+	)
+	(gr_rect
+		(start 95.8 100.9)
+		(end 110.1 115.9)
+		(stroke
+			(width 0.1)
+			(type default)
+		)
+		(fill none)
+		(layer "User.2")
 	)
 	(gr_rect
@@
 	)
 	(gr_rect
-		(start 126.9 100.9)
-		(end 141.2 115.9)
-		(stroke
-			(width 0.1)
-			(type default)
-		)
-		(fill none)
-		(layer "User.2")
-	)
-	(gr_rect
-		(start 216.5 100.9)
-		(end 230.8 115.9)
-		(stroke
-			(width 0.1)
-			(type default)
-		)
-		(fill none)
-		(layer "User.2")
-	)
-	(gr_rect
-		(start 141.2 100.9)
-		(end 155.5 115.9)
-		(stroke
-			(width 0.1)
-			(type default)
-		)
-		(fill none)
-		(layer "User.2")
-	)
-	(gr_rect
-		(start 95.8 100.9)
-		(end 110.1 115.8)
-		(stroke
-			(width 0.1)
-			(type default)
-		)
-		(fill none)
-		(layer "User.2")
-	)
-	(gr_rect
-		(start 187.9 101)
-		(end 202.2 115.9)
-		(stroke
-			(width 0.1)
-			(type default)
-		)
-		(fill none)
-		(layer "User.2")
-	)
-	(gr_rect
-		(start 112.6 101)
-		(end 126.9 115.9)
-		(stroke
-			(width 0.1)
-			(type default)
-		)
-		(fill none)
-		(layer "User.2")
-	)
-	(gr_rect
-		(start 169.8 100.9)
-		(end 184.1 115.9)
-		(stroke
-			(width 0.1)
-			(type default)
-		)
-		(fill none)
-		(layer "User.2")
-	)
-	(gr_rect
-		(start 155.5 101)
-		(end 169.8 115.9)
+		(start 201.8 100.9)
+		(end 216.1 115.9)
+		(stroke
+			(width 0.1)
+			(type default)
+		)
+		(fill none)
+		(layer "User.2")
+	)
+	(gr_rect
+		(start 187.5 100.9)
+		(end 201.8 115.9)
+		(stroke
+			(width 0.1)
+			(type default)
+		)
+		(fill none)
+		(layer "User.2")
+	)
+	(gr_rect
+		(start 127.1 100.9)
+		(end 141.6 115.9)
 		(stroke
 			(width 0.1)
@@
 	)
 	(gr_rect
-		(start 202.2 100.9)
-		(end 216.5 115.9)
-		(stroke
-			(width 0.1)
-			(type default)
-		)
-		(fill none)
-		(layer "User.2")
-	)
-	(zone
-		(net 0)
-		(net_name "")
-		(layer "User.1")
-		(hatch edge 0.5)
-		(connect_pads
-			(clearance 0.5)
-		)
-		(min_thickness 0.25)
-		(filled_areas_thickness no)
-		(fill yes
-			(thermal_gap 0.5)
-			(thermal_bridge_width 0.5)
-		)
-		(polygon
-			(pts
-				(xy 110.2 100.9) (xy 112.6 100.9) (xy 112.6 115.9) (xy 110.2 115.9)
-			)
-		)
-	)
-	(zone
-		(net 0)
-		(net_name "")
-		(layer "User.1")
-		(hatch edge 0.5)
-		(connect_pads
-			(clearance 0.5)
-		)
-		(min_thickness 0.25)
-		(filled_areas_thickness no)
-		(fill yes
-			(thermal_gap 0.5)
-			(thermal_bridge_width 0.5)
-		)
-		(polygon
-			(pts
-				(xy 185.6 100.9) (xy 188 100.9) (xy 188 115.9) (xy 185.6 115.9)
-			)
-		)
-	)
-	(zone
-		(net 0)
-		(net_name "")
-		(layer "User.1")
-		(hatch edge 0.5)
-		(connect_pads
-			(clearance 0.5)
-		)
-		(min_thickness 0.25)
-		(filled_areas_thickness no)
-		(fill yes
-			(thermal_gap 0.5)
-			(thermal_bridge_width 0.5)
-		)
-		(polygon
-			(pts
-				(xy 67.2 92.3) (xy 236.2 92.3) (xy 236.2 100.9) (xy 67.2 100.9)
-			)
-		)
+		(start 156.1 100.9)
+		(end 170.6 115.9)
+		(stroke
+			(width 0.1)
+			(type default)
+		)
+		(fill none)
+		(layer "User.2")
+	)
+	(gr_rect
+		(start 141.6 100.9)
+		(end 156.1 115.9)
+		(stroke
+			(width 0.1)
+			(type default)
+		)
+		(fill none)
+		(layer "User.2")
+	)
+	(gr_rect
+		(start 112.6 100.9)
+		(end 127.1 115.9)
+		(stroke
+			(width 0.1)
+			(type default)
+		)
+		(fill none)
+		(layer "User.2")
+	)
+	(gr_rect
+		(start 216.1 100.9)
+		(end 230.4 115.9)
+		(stroke
+			(width 0.1)
+			(type default)
+		)
+		(fill none)
+		(layer "User.2")
+	)
+	(gr_rect
+		(start 112.6 100.9)
+		(end 185.1 115.9)
+		(stroke
+			(width 0.1)
+			(type default)
+		)
+		(fill none)
+		(layer "User.3")
+	)
+	(gr_rect
+		(start 67.2 100.9)
+		(end 110.2 115.9)
+		(stroke
+			(width 0.1)
+			(type default)
+		)
+		(fill none)
+		(layer "User.3")
+	)
+	(gr_rect
+		(start 187.5 100.9)
+		(end 230.5 115.9)
+		(stroke
+			(width 0.1)
+			(type default)
+		)
+		(fill none)
+		(layer "User.3")
 	)
 )
