File: ErrorDisplay/ErrorDisplay/CANBus.kicad_sch (KiCad schematic)
At the start: 2 parts, among them U1 MCP2562-E-SN

Commit message: WIP checkin
Changed lines of the file:
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@@
+		)
+	)
+	(label "CAN_TXD"
+		(at 273.05 19.05 180)
+		(fields_autoplaced yes)
+		(effects
+			(font
+				(size 1.27 1.27)
+			)
+			(justify right bottom)
 		)
 	)
@@
 		)
 	)
+	(label "CAN_RXD"
+		(at 273.05 21.59 180)
+		(fields_autoplaced yes)
+		(effects
+			(font
+				(size 1.27 1.27)
+			)
+			(justify right bottom)
+		)
+	)
 	(label "CAN_STBY"
 		(at 24.13 22.86 0)
@@
 			)
 			(justify left bottom)
+		)
+	)
+	(hierarchical_label "CAN_RXD"
+		(shape input)
+		(at 273.05 21.59 0)
+		(fields_autoplaced yes)
+		(effects
+			(font
+				(size 1.27 1.27)
+			)
+			(justify left)
 		)
 	)
@@
 		)
 	)
+	(hierarchical_label "CAN_TXD"
+		(shape input)
+		(at 273.05 19.05 0)
+		(fields_autoplaced yes)
+		(effects
+			(font
+				(size 1.27 1.27)
+			)
+			(justify left)
+		)
+	)
