File: ErrorDisplay/ErrorDisplay/DigitalDisplay.kicad_sch (KiCad schematic)
At the start: 12 parts, among them J5 Conn_01x01_Pin

Commit message: WIP checkin
Parts:
- added C2: 0.1u, Capacitor_SMD:C_0402_1005Metric_Pad0.74x0.62mm_HandSolder, symbol Device:C
- added R1, R2: 100k, Resistor_SMD:R_0402_1005Metric_Pad0.72x0.64mm_HandSolder, symbol Device:R
- added R10, R11, R12, R13, R14, R15, R16, R3, R4, R6, R7, R8, R9: R, Resistor_SMD:R_0402_1005Metric_Pad0.72x0.64mm_HandSolder, symbol Device:R
- added R5: 0, Resistor_SMD:R_0402_1005Metric_Pad0.72x0.64mm_HandSolder, symbol Device:R
- added U2: MCP23017_SS, Package_SO:SSOP-28_5.3x10.2mm_P0.65mm, symbol Interface_Expansion:MCP23017_SS
Connections:
- net GND: now also 12V_LED1.1 (K), BR_LED1.1 (K), DEFROST_LED1.1 (K), ERR_LED1.1 (K), HV_LED1.1 (K), LEFT_LED1.1 (K), LIGHT_LED1.1 (K), MOT_TEMP_LED1.2 (K), PARK_LED1.1 (K), RIGHT_LED1.1 (K), TEMP_LED1.2 (K), C2.2, R2.2, U2.10 (VSS), U2.15 (A0), U2.16 (A1), U2.17 (A2)
- net at LIGHT_LED1.2 (A): now also R11.2
- net at HV_LED1.2 (A): now also R8.2
- net at TEMP_LED1.1 (A1): now also R6.2
- net at TEMP_LED1.3 (A2): now also R7.2
- net at DEFROST_LED1.2 (A): now also R15.2
- net at RIGHT_LED1.2 (A): now also R14.2
- net at MOT_TEMP_LED1.1 (A1): now also R3.2
- net at MOT_TEMP_LED1.3 (A2): now also R4.2
- net at ERR_LED1.2 (A): now also R9.2
- net at LEFT_LED1.2 (A): now also R12.2
- net at PARK_LED1.2 (A): now also R13.2
- net at 12V_LED1.2 (A): now also R16.2
- net at BR_LED1.2 (A): now also R10.2
- new net: R1.2, R2.1, U2.18 (~{RESET})
- new net +5V: R5.1
- new net 12VLED: R16.1, U2.25 (GPA4)
- new net BRIGHTLED: R10.1, U2.7 (GPB6)
- new net CONT_A: R7.1, U2.4 (GPB3)
- new net CONT_R: R6.1, U2.3 (GPB2)
- new net DEFROSTLED: R15.1, U2.24 (GPA3)
- new net ERRLED: R9.1, U2.6 (GPB5)
- new net HVLED: R8.1, U2.5 (GPB4)
- new net LEFTLED: R12.1, U2.21 (GPA0)
- new net LIGHTLED: R11.1, U2.8 (GPB7)
- new net MOT_A: R4.1, U2.2 (GPB1)
- new net MOT_R: R3.1, U2.1 (GPB0)
- new net PARKLED: R13.1, U2.22 (GPA1)
- new net RIGHTLED: R14.1, U2.23 (GPA2)
- new net SCL: U2.12 (SCK)
- new net SDA: U2.13 (SDA)
- new net VLED: C2.1, R1.1, R5.2, U2.9 (VDD)
- no-connect marks 0 -> 5
Other:
- moved on the sheet: 12V_LED1
