File: ErrorDisplay/ErrorDisplay/Power.kicad_sch (KiCad schematic)
At the start: 0 parts

Commit message: WIP checkin
Parts:
- added C3, C5: 4.7u, Capacitor_SMD:C_0603_1608Metric, symbol Device:C
- added C4: 100n, Capacitor_SMD:C_0603_1608Metric, symbol Device:C
- added D2, D3, D4: LED, LED_SMD:LED_0603_1608Metric_Pad1.05x0.95mm_HandSolder, symbol Device:LED
- added JP1: Jumper_2_Open, Resistor_SMD:R_0805_2012Metric, symbol Jumper:Jumper_2_Open
- added L1: 12u, Inductor_SMD:L_1812_4532Metric, symbol Device:L
- added R18: 0, Resistor_SMD:R_0402_1005Metric_Pad0.72x0.64mm_HandSolder, symbol Device:R
- added R19, R22: 4.7k, Resistor_SMD:R_0402_1005Metric_Pad0.72x0.64mm_HandSolder, symbol Device:R
- added R20: 100k, Resistor_SMD:R_0402_1005Metric, symbol Device:R
- added R21: 15.4k, Resistor_SMD:R_0402_1005Metric, symbol Device:R
- added U3: MIC5365-3.3YC5, Package_TO_SOT_SMD:SOT-353_SC-70-5, symbol Regulator_Linear:MIC5365-3.3YC5
- added U4: TPS54308, Package_TO_SOT_SMD:SOT-23-6, symbol Regulator_Switching:TPS54308
Connections:
- net CAN_VCC: now also D2.2 (A), JP1.1 (A), U4.3 (VIN), U4.5 (EN)
- new net: D3.1 (K), R19.1
- new net: C4.1, U4.6 (BOOT)
- new net: C4.2, L1.1, U4.2 (SW)
- new net: R20.2, R21.1, U4.4 (FB)
- new net: D2.1 (K), R18.1
- new net: D4.1 (K), R22.1
- new net +3V3: C3.1, D3.2 (A), U3.5 (VOUT)
- new net +5V: C5.1, D4.2 (A), JP1.2 (B), L1.2, R20.1, U3.1 (VIN), U3.3 (EN)
- new net GND: C3.2, C5.2, R18.2, R19.2, R21.2, R22.2, U3.2 (GND), U4.1 (GND)
Other:
- note added: "TODO"
- note added: "TODO untested. SeeTestbed1"
