File: MainController/VoltageMeasurement.kicad_sch (KiCad schematic)
At the start: 7 parts

Commit message: WIP - HV measurement may be done
Parts:
- added C11, C13: 0.1u, Capacitor_SMD:C_0402_1005Metric_Pad0.74x0.62mm_HandSolder, symbol Device:C
- added C12, C14: 1u, Capacitor_SMD:C_0402_1005Metric_Pad0.74x0.62mm_HandSolder, symbol Device:C
- R3: value R -> 0
Connections:
- net +3V3: now also C13.1, C14.1
- net GND: now also U2.5 (GND2), C13.2, C14.2
- net 3v3_iso: now reaches U2.1 (VDD1)
- net 3v3_iso: now also C11.1, C12.1
- net OUTN: now reaches U2.6 (OUTN)
- net OUTP: now reaches U2.7 (OUTP)
- net HV_IN_- renamed GND1
- net GND1: now also C11.2, C12.2
Other:
- note removed: "TODO Use B? Likely need to buck HV down. If need to buck down 80V to low voltage, 5V is fine."
- note removed: "TODO can I use an optoisolater to give the high side? Can use an isolated output. Maybe enough current? Check datasheet"
