File: BenchTest/BenchTest2_MIC4606/BenchTest2_MIC4606/HBridgeDriver.kicad_sch (KiCad schematic)
At the start: 39 parts, among them J1 Conn_01x01_Socket, J2 Conn_01x01_Socket, J3 Conn_01x01_Socket, J4 Conn_01x01_Socket, J5 Conn_01x01_Socket, J6 Conn_01x01_Socket, J7 Conn_01x01_Socket, J8 Conn_01x01_Socket

Commit message: Board to ship for Fets
Parts:
- C1: footprint Capacitor_SMD:C_0603_1608Metric_Pad1.08x0.95mm_HandSolder -> Capacitor_SMD:C_0402_1005Metric_Pad0.74x0.62mm_HandSolder
- C3: value 4.7u -> 2.2u
Changed lines of the file:
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@@
 		)
 	)
-	(label "G2"
-		(at 246.38 111.76 180)
+	(label "Vdrive"
+		(at 22.86 17.78 0)
 		(fields_autoplaced yes)
 		(effects
@@
 				(size 1.27 1.27)
 			)
-			(justify right bottom)
-		)
-	)
-	(label "Vdrive"
-		(at 63.5 156.21 90)
+			(justify left bottom)
+		)
+	)
+	(label "G2"
+		(at 246.38 111.76 180)
 		(fields_autoplaced yes)
 		(effects
@@
 				(size 1.27 1.27)
 			)
-			(justify left bottom)
+			(justify right bottom)
 		)
 	)
 	(label "Vdrive"
-		(at 90.17 135.89 90)
+		(at 63.5 156.21 90)
 		(fields_autoplaced yes)
 		(effects
@@
 		)
 	)
-	(label "G3"
-		(at 123.19 96.52 180)
+	(label "Vdrive"
+		(at 90.17 135.89 90)
 		(fields_autoplaced yes)
 		(effects
@@
 				(size 1.27 1.27)
 			)
-			(justify right bottom)
-		)
-	)
-	(label "Motor0"
-		(at 144.78 81.28 180)
+			(justify left bottom)
+		)
+	)
+	(label "G3"
+		(at 123.19 96.52 180)
 		(fields_autoplaced yes)
 		(effects
@@
 		)
 	)
-	(label "APWM"
-		(at 73.66 144.78 180)
+	(label "Motor0"
+		(at 144.78 81.28 180)
 		(fields_autoplaced yes)
 		(effects
@@
 		)
 	)
-	(label "ALO"
-		(at 105.41 149.86 0)
+	(label "APWM"
+		(at 73.66 144.78 180)
 		(fields_autoplaced yes)
 		(effects
@@
 				(size 1.27 1.27)
 			)
-			(justify left bottom)
-		)
-	)
-	(label "AHB"
-		(at 105.41 140.97 0)
+			(justify right bottom)
+		)
+	)
+	(label "ALO"
+		(at 105.41 149.86 0)
 		(fields_autoplaced yes)
 		(effects
@@
 		)
 	)
-	(label "APWM"
-		(at 179.07 144.78 180)
+	(label "AHB"
+		(at 105.41 140.97 0)
 		(fields_autoplaced yes)
 		(effects
@@
 				(size 1.27 1.27)
 			)
-			(justify right bottom)
-		)
-	)
-	(label "G4"
-		(at 167.64 96.52 180)
+			(justify left bottom)
+		)
+	)
+	(label "APWM"
+		(at 179.07 144.78 180)
 		(fields_autoplaced yes)
 		(effects
@@
 	)
 	(label "G4"
-		(at 246.38 124.46 180)
+		(at 167.64 96.52 180)
 		(fields_autoplaced yes)
 		(effects
@@
 		)
 	)
-	(label "Vdrive"
-		(at 44.45 156.21 90)
+	(label "G4"
+		(at 246.38 124.46 180)
 		(fields_autoplaced yes)
 		(effects
@@
 				(size 1.27 1.27)
 			)
-			(justify left bottom)
+			(justify right bottom)
 		)
 	)
 	(label "Vdrive"
-		(at 68.58 132.08 90)
+		(at 44.45 156.21 90)
 		(fields_autoplaced yes)
 		(effects
@@
 		)
 	)
-	(label "G2"
-		(at 167.64 67.31 0)
+	(label "Vdrive"
+		(at 68.58 132.08 90)
 		(fields_autoplaced yes)
 		(effects
@@
 		)
 	)
-	(label "BPWM"
-		(at 73.66 148.59 180)
+	(label "G2"
+		(at 167.64 67.31 0)
 		(fields_autoplaced yes)
 		(effects
@@
 				(size 1.27 1.27)
 			)
-			(justify right bottom)
+			(justify left bottom)
 		)
 	)
 	(label "BPWM"
-		(at 179.07 149.86 180)
+		(at 73.66 148.59 180)
 		(fields_autoplaced yes)
 		(effects
@@
 		)
 	)
-	(label "BHB"
-		(at 105.41 162.56 0)
+	(label "BPWM"
+		(at 179.07 149.86 180)
 		(fields_autoplaced yes)
 		(effects
@@
 				(size 1.27 1.27)
 			)
-			(justify left bottom)
-		)
-	)
-	(label "AHS"
-		(at 105.41 146.05 0)
+			(justify right bottom)
+		)
+	)
+	(label "BHB"
+		(at 105.41 162.56 0)
 		(fields_autoplaced yes)
 		(effects
@@
 		)
 	)
+	(label "AHS"
+		(at 105.41 146.05 0)
+		(fields_autoplaced yes)
+		(effects
+			(font
+				(size 1.27 1.27)
+			)
+			(justify left bottom)
+		)
+	)
+	(hierarchical_label "Vdrive"
+		(shape input)
+		(at 22.86 17.78 180)
+		(fields_autoplaced yes)
+		(effects
+			(font
+				(size 1.27 1.27)
+			)
+			(justify right)
+		)
+	)
 	(symbol
 		(lib_id "Device:C")
@@
 			)
 		)
-		(property "Value" "4.7u"
+		(property "Value" "2.2u"
 			(at 66.421 161.2321 0)
 			(effects
@@
 			)
 		)
-		(property "Footprint" "Capacitor_SMD:C_0603_1608Metric_Pad1.08x0.95mm_HandSolder"
+		(property "Footprint" "Capacitor_SMD:C_0402_1005Metric_Pad0.74x0.62mm_HandSolder"
 			(at 45.4152 163.83 0)
 			(effects
