File: BenchTest/BenchTest2_MIC4606/BenchTest2_MIC4606/Regen.kicad_sch (KiCad schematic)
At the start: 15 parts, among them Q3 Q_PMOS_DGS, Q4 Q_PMOS_DGS, U4 TLP2767

Commit message: H Bridge Continuation
Other:
- note added: "TODO is this PFET?"
Changed lines of the file:
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@@
 	(generator_version "9.0")
 	(paper "A4")
+	(text "TODO is this PFET?"
+		(exclude_from_sim no)
+		(at 248.92 83.566 0)
+		(effects
+			(font
+				(size 1.27 1.27)
+			)
+		)
+	)
 	(text "TODO > 100v reverse schotkey"
 		(exclude_from_sim no)
