File: BenchTest/BenchTest2_MIC4606/BenchTest2_MIC4606/MotorConnection .kicad_sch (KiCad schematic)
At the start: 4 parts, among them J1 Conn_01x01_Socket, J2 Conn_01x03, J3 Conn_01x01_Socket, J4 Conn_01x01_Socket

Commit message: Additional Documents / Routing
Parts:
- removed J2: Conn_01x03, symbol Connector_Generic:Conn_01x03
- added J5: Conn_01x01_Socket, symbol Connector:Conn_01x01_Socket
Connections:
- new net MOTORCON+: J5.1 (Pin_1)
Other:
- note removed: "TODO add Hall sensor connector footprint"
- moved on the sheet: J1
Changed lines of the file:
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@@
-		)
-	)
-	(text "TODO add Hall sensor connector footprint"
-		(exclude_from_sim no)
-		(at 193.548 49.784 0)
-		(effects
-			(font
-				(size 1.27 1.27)
-			)
 		)
 	)
 	(text "TODO which footprint"
 		(exclude_from_sim no)
-		(at 234.696 58.42 0)
+		(at 195.326 76.2 0)
 		(effects
 			(font
@@
 	(text "TODO which footprint"
 		(exclude_from_sim no)
+		(at 234.442 77.724 0)
+		(effects
+			(font
+				(size 1.27 1.27)
+			)
+		)
+	)
+	(text "TODO design for > 100A"
+		(exclude_from_sim no)
+		(at 235.966 75.438 0)
+		(effects
+			(font
+				(size 1.27 1.27)
+			)
+		)
+	)
+	(text "TODO which footprint"
+		(exclude_from_sim no)
 		(at 215.646 132.08 0)
 		(effects
@@
 	(text "TODO design for > 100A"
 		(exclude_from_sim no)
-		(at 235.458 55.88 0)
+		(at 196.088 73.66 0)
 		(effects
 			(font
@@
 		)
 	)
-	(label "current_sns"
+	(label "Mot+"
 		(at 269.24 19.05 180)
 		(effects
@@
 		)
 	)
-	(label "vdrive"
-		(at 176.53 55.88 180)
+	(label "Mot+"
+		(at 234.95 85.09 270)
 		(effects
 			(font
@@
 	)
 	(label "Mot-"
-		(at 234.95 67.31 270)
+		(at 195.58 85.09 270)
 		(effects
 			(font
@@
 	(label "F1"
 		(at 279.4 31.75 180)
-		(effects
-			(font
-				(size 1.27 1.27)
-			)
-			(justify right bottom)
-		)
-	)
-	(label "current_sns"
-		(at 185.42 60.96 180)
 		(effects
 			(font
@@
 		)
 	)
-	(hierarchical_label "CURRENT_SNS"
+	(hierarchical_label "MOTORCON+"
 		(shape input)
 		(at 269.24 19.05 0)
@@
 	(symbol
 		(lib_id "Connector:Conn_01x01_Socket")
-		(at 234.95 62.23 90)
+		(at 195.58 80.01 90)
 		(unit 1)
 		(exclude_from_sim no)
@@
 		(fields_autoplaced yes)
 		(property "Reference" "J1"
-			(at 236.22 61.5949 90)
+			(at 196.85 79.3749 90)
 			(effects
 				(font
@@
 		)
 		(property "Value" "Conn_01x01_Socket"
-			(at 236.22 64.1349 90)
+			(at 196.85 81.9149 90)
 			(effects
 				(font
@@
 		)
 		(property "Footprint" ""
-			(at 234.95 62.23 0)
+			(at 195.58 80.01 0)
 			(effects
 				(font
@@
 		)
 		(property "Datasheet" "~"
-			(at 234.95 62.23 0)
+			(at 195.58 80.01 0)
 			(effects
 				(font
@@
 		)
 		(property "Description" "Generic connector, single row, 01x01, script generated"
-			(at 234.95 62.23 0)
+			(at 195.58 80.01 0)
 			(effects
 				(font
@@
 	)
 	(symbol
-		(lib_id "Connector_Generic:Conn_01x03")
-		(at 196.85 60.96 0)
+		(lib_id "Connector:Conn_01x01_Socket")
+		(at 234.95 80.01 90)
 		(unit 1)
 		(exclude_from_sim no)
@@
 		(dnp no)
 		(fields_autoplaced yes)
-		(property "Reference" "J2"
-			(at 199.39 59.6899 0)
-			(effects
-				(font
-					(size 1.27 1.27)
-				)
-				(justify left)
-			)
-		)
-		(property "Value" "Conn_01x03"
-			(at 199.39 62.2299 0)
-			(effects
-				(font
-					(size 1.27 1.27)
-				)
-				(justify left)
+		(property "Reference" "J5"
+			(at 236.22 79.3749 90)
+			(effects
+				(font
+					(size 1.27 1.27)
+				)
+				(justify right)
+			)
+		)
+		(property "Value" "Conn_01x01_Socket"
+			(at 236.22 81.9149 90)
+			(effects
+				(font
+					(size 1.27 1.27)
+				)
+				(justify right)
 			)
 		)
 		(property "Footprint" ""
-			(at 196.85 60.96 0)
+			(at 234.95 80.01 0)
 			(effects
 				(font
@@
 		)
 		(property "Datasheet" "~"
-			(at 196.85 60.96 0)
-			(effects
-				(font
-					(size 1.27 1.27)
-				)
-				(hide yes)
-			)
-		)
-		(property "Description" "Generic connector, single row, 01x03, script generated (kicad-library-utils/schlib/autogen/connector/)"
-			(at 196.85 60.96 0)
+			(at 234.95 80.01 0)
+			(effects
+				(font
+					(size 1.27 1.27)
+				)
+				(hide yes)
+			)
+		)
+		(property "Description" "Generic connector, single row, 01x01, script generated"
+			(at 234.95 80.01 0)
 			(effects
 				(font
@@
 		)
 		(pin "1"
-		)
-		(pin "2"
-		)
-		(pin "3"
 		)
 		(instances
 			(project "BenchTest2_MIC4606"
 				(path "/5c5197d3-4aa5-4f8b-b790-1e4b8d49fd62/592b72e5-95a7-493e-b4e9-fc1a8b0156f6"
-					(reference "J2")
+					(reference "J5")
 					(unit 1)
 				)
@@
 					(unit 1)
 				)
-			)
-		)
-	)
-	(symbol
-		(lib_id "power:GND")
-		(at 182.88 72.39 0)
-		(unit 1)
-		(exclude_from_sim no)
-		(in_bom yes)
-		(on_board yes)
-		(dnp no)
-		(fields_autoplaced yes)
-		(property "Reference" "#PWR01"
-			(at 182.88 78.74 0)
-			(effects
-				(font
-					(size 1.27 1.27)
-				)
-				(hide yes)
-			)
-		)
-		(property "Value" "GND"
-			(at 182.88 77.47 0)
-			(effects
-				(font
-					(size 1.27 1.27)
-				)
-			)
-		)
-		(property "Footprint" ""
-			(at 182.88 72.39 0)
-			(effects
-				(font
-					(size 1.27 1.27)
-				)
-				(hide yes)
-			)
-		)
-		(property "Datasheet" ""
-			(at 182.88 72.39 0)
-			(effects
-				(font
-					(size 1.27 1.27)
-				)
-				(hide yes)
-			)
-		)
-		(property "Description" "Power symbol creates a global label with name \"GND\" , ground"
-			(at 182.88 72.39 0)
-			(effects
-				(font
-					(size 1.27 1.27)
-				)
-				(hide yes)
-			)
-		)
-		(pin "1"
-		)
-		(instances
-			(project ""
-				(path "/5c5197d3-4aa5-4f8b-b790-1e4b8d49fd62/592b72e5-95a7-493e-b4e9-fc1a8b0156f6"
-					(reference "#PWR01")
-					(unit 1)
-				)
