File: BenchTest/BenchTest2_MIC4606/BenchTest2_MIC4606/BenchTest2_MIC4606.kicad_pcb (KiCad board)
At the start: 2 copper layers, 50.5 x 59.5 mm, 55 parts, among them J1 Conn_01x01_Socket, J10 Conn_01x01_Socket, J11 Conn_01x01_Socket, J12 Conn_01x01_Socket, J13 Conn_01x01_Socket, J14 Conn_01x01_Socket, J15 Conn_01x01_Socket, J2 Conn_01x01_Socket, J3 Conn_01x01_Socket, J4 Conn_01x01_Socket, J5 Conn_01x01_Socket, J6 Conn_01x01_Socket, J7 Conn_01x01_Socket, J8 Conn_01x01_Socket, J9 Conn_01x02_Socket

Commit message: Footprint / Capacitor Assignment
Parts:
- removed C1, C10, C12: 0.1u, Capacitor_SMD:C_0402_1005Metric_Pad0.74x0.62mm_HandSolder
- removed C11, C13, C3: 2.2u, Capacitor_SMD:C_0603_1608Metric_Pad1.08x0.95mm_HandSolder
- removed C2: 1u, Capacitor_SMD:C_0603_1608Metric_Pad1.08x0.95mm_HandSolder
- removed C4, C5, C8, C9: 4.7n, Capacitor_SMD:C_0805_2012Metric_Pad1.18x1.45mm_HandSolder
- removed C6, C7: 10u, Capacitor_SMD:C_0805_2012Metric_Pad1.18x1.45mm_HandSolder
- removed D1, D2, D3, D4, D5, D6: D, Diode_SMD:D_SOD-123F
- removed J1, J10, J11, J12, J13, J14, J15, J2, J3, J4, J5, J6, J7, J8: Conn_01x01_Socket, Connector_PinHeader_2.54mm:PinHeader_1x01_P2.54mm_Vertical
- removed J9: Conn_01x02_Socket, Connector_PinHeader_2.54mm:PinHeader_1x02_P2.54mm_Vertical
- removed R1: 100k, Resistor_SMD:R_0402_1005Metric_Pad0.72x0.64mm_HandSolder
- removed R10, R2, R5, R9: 6.8, Resistor_SMD:R_0805_2012Metric_Pad1.20x1.40mm_HandSolder
- removed R11, R3, R4, R8: 18, Resistor_SMD:R_0805_2012Metric_Pad1.20x1.40mm_HandSolder
- removed R12, R13, R14: 33, Resistor_SMD:R_0402_1005Metric_Pad0.72x0.64mm_HandSolder
- removed R6, R7: 3.3, Resistor_SMD:R_0805_2012Metric_Pad1.20x1.40mm_HandSolder
- removed TP1, TP2, TP3, TP4: TestPoint, TestPoint:TestPoint_Pad_1.0x1.0mm
- removed U1: ~, Package_SO:TSSOP-16_4.4x5mm_P0.65mm
- removed U2, U3: ~, Package_SO:SOIC-8_3.9x4.9mm_P1.27mm
Routing:
- net /Vdrive: track 120.7 -> 0.00 mm, vias 4 -> 0
- net /HBridgeDriver/BHB: track 55.8 -> 0.00 mm, vias 4 -> 0
- net /HBridgeDriver/BHS: track 36.3 -> 0.00 mm
- net /HBridgeDriver/G2: track 31.9 -> 0.00 mm
- net /HBridgeDriver/ALO: track 27.4 -> 0.00 mm
- net /HBridgeDriver/G1: track 26.6 -> 0.00 mm, vias 2 -> 0
- net /HBridgeDriver/BHO: track 22.2 -> 0.00 mm
- net GND: track 21.4 -> 0.00 mm, vias 11 -> 0
- net /HBridgeDriver/AHO: track 19.9 -> 0.00 mm, vias 2 -> 0
- net /HBridgeDriver/BLO: track 18.9 -> 0.00 mm
- net /G6: track 14.0 -> 0.00 mm
- net /HBridgeDriver/Motor0: track 13.9 -> 0.00 mm
- net /HBridgeDriver/AHB: track 12.4 -> 0.00 mm, vias 2 -> 0
- net /HBridgeDriver/AHS: track 12.0 -> 0.00 mm
- net /HBridgeDriver/G3: track 12.0 -> 0.00 mm
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- removed copper zone on B.Cu, net GND
Other:
- board outline removed
