File: BenchTest/Controller/ExternalConnections.kicad_sch (KiCad schematic)
At the start: 0 parts

Commit message: Added Isolation for digital drives
Other:
- note added: "TODO Pedal Connection"
Changed lines of the file:
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@@
 	(generator_version "9.0")
 	(paper "A4")
+	(text "TODO Pedal Connection"
+		(exclude_from_sim no)
+		(at 205.232 66.802 0)
+		(effects
+			(font
+				(size 1.27 1.27)
+			)
+		)
+	)
 )

Commit message: WIP Controller in progress
w
Parts:
- added J5: Conn_01x04, symbol Connector_Generic:Conn_01x04
Connections:
- new net +3V3: J5.1 (Pin_1)
- new net GND: J5.4 (Pin_4)
- new net LED_MOSI: J5.2 (Pin_2)
- new net LED_SCK: J5.3 (Pin_3)
Other:
- note removed: "TODO Pedal Connection"
